Commit message: urdf: wheel radius 0.049 -> 0.050 to match the firmware default
VISUAL ONLY - odometry was never affected. driver.py reads kin.wheel_radius from
the board at start-up (line 92) and uses the live value, so the maths was always
correct and self-updating. The URDF cylinders are what RViz draws.

Fixing it anyway because a hard-coded constant that disagrees with the board by
2 percent looks authoritative to the next reader, and this one had already
survived the 1.14.1 firmware change unnoticed.

Co-Authored-By: Claude Opus 5 <noreply@anthropic.com>

File: src/orcp_ros2/urdf/orcp_bot.urdf (robot description, URDF)
Before this commit: robot orcp_bot, 3 links, 2 joints
Links:
- link left_wheel: geometry visual cylinder length=0.02 radius=0.050
- link right_wheel: geometry visual cylinder length=0.02 radius=0.050
